File: KiCad/ardHoneyServo/ardHoneyServo.kicad_pcb (KiCad board)
At the start: 2 copper layers, 62.2 x 56.5 mm, 14 parts, among them J1 LCD, K1 Spinner motor, M1 Servo, U1 Buttons / Switches, U2 Rotary encoder

Commit message: pcb
Other:
- board text added: "ardHoneyServo-0.1 Design: Jon Sagebrand github.com/jonsag"
Changed lines of the file:
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@@
   (gr_line (start 180.34 71.12) (end 183.515 73.66) (layer "Edge.Cuts") (width 0.1))
   (gr_line (start 121.285 56.515) (end 177.165 56.515) (layer "Edge.Cuts") (width 0.1))
+  (gr_text "ardHoneyServo-0.1\nDesign: Jon Sagebrand\ngithub.com/jonsag" (at 173.99 78.105 90) (layer "B.Cu")
+    (effects (font (size 0.889 0.889) (thickness 0.22225)) (justify left mirror))
+  )
   (segment (start 146.05 76.835) (end 149.928707 80.713707) (width 0.762) (layer "F.Cu") (net 5))
   (segment (start 151.5225 88.6575) (end 151.5225 84.561463) (width 0.762) (layer "F.Cu") (net 5))
