File: KiCad/ardHoneyServo/ardHoneyServo.kicad_sch (KiCad schematic)
At the start: 14 parts, among them J1 LCD, K1 Spinner motor, M1 Servo, U1 Buttons / Switches, U2 Rotary encoder

Commit message: kicad7
Other:
- title: (none) -> ardHoneyServo
